Commit message: slam_integration

File: description/robotie.xacro (robot description, xacro)
@@ -6,4 +6,11 @@
     <xacro:include filename="ros2_control.xacro"/>
     <link name="base_link"/>
+    <link name="base_footprint">
+    </link>
+    <joint name="base_footprint_joint" type="fixed">
+        <origin xyz="0.0 0.0 0.0" rpy="0.0 0.0 0.0"/>
+        <parent link="base_link"/>
+        <child link="base_footprint"/>
+    </joint>
     <joint name="chassis_joint" type="fixed">
         <parent link="base_link"/>
