Commit message: ro2_control

File: description/gazebo.xacro (robot description, xacro)
@@ -87,5 +87,5 @@
             <plugin name="laser_controller" filename="libgazebo_ros_ray_sensor.so">
                 <ros>
-                    <argument>~/out:=scan</argument>
+                    <argument>out:=scan</argument>
                 </ros>
                 <output_type>sensor_msgs/LaserScan</output_type>

File: description/robotie.xacro (robot description, xacro)
@@ -4,4 +4,5 @@
     <xacro:include filename="properties.xacro"/>
     <xacro:include filename="gazebo.xacro"/>
+    <xacro:include filename="ros2_control.xacro"/>
     <link name="base_link"/>
     <joint name="chassis_joint" type="fixed">
@@ -33,5 +34,4 @@
         <origin xyz="0 ${wheel_offset_y} 0" rpy="-${pi/2} 0 0" />
         <axis xyz="0 0 1"/>
-        <dynamics damping="0.7" friction="0.2"/>
     </joint>
     <link name="left_wheel">
@@ -56,5 +56,4 @@
         <origin xyz="0 ${-wheel_offset_y} 0" rpy="${pi/2} 0 0" />
         <axis xyz="0 0 -1"/>
-        <dynamics damping="0.7" friction="0.2"/>
     </joint>
     <link name="right_wheel">

Commit message: diff_controller

File: description/gazebo.xacro (robot description, xacro)
@@ -22,5 +22,5 @@
     <gazebo reference="caster_wheel">
         <material>
-            Gazebo/White
+            Gazebo/Black
         </material>
         <mu1>0.02</mu1>

File: description/properties.xacro (robot description, xacro)
@@ -12,5 +12,5 @@
     <xacro:property name="wheel_offset_z" value="0.01"/>
     <xacro:property name="caster_wheel_radius" value="0.05"/>
-    <xacro:property name="caster_wheel_mass" value="0.01"/>
+    <xacro:property name="caster_wheel_mass" value="0.5"/>
     <xacro:property name="caster_wheel_offset_x" value="0.075"/>
     <xacro:property name="caster_wheel_offset_z" value="${wheel_offset_z - wheel_radius + caster_wheel_radius}"/>

Commit message: lidar_fixes

File: description/gazebo.xacro (robot description, xacro)
@@ -61,10 +61,10 @@
         </sensor>
     </gazebo>
-    <gazebo reference="hokuyo_base_link">
+    <gazebo reference="lidar_base_link">
         <material>
             Gazebo/Black
         </material>
     </gazebo>
-    <gazebo reference="hokuyo_link">
+    <gazebo reference="lidar_link">
         <material>Gazebo/Black</material>
         <sensor name="laser" type="ray">
@@ -85,10 +85,10 @@
                 </range>
             </ray>
-            <plugin name="laser_controller" filename="libgazebo_ros_ray_sensor.so">
+             <plugin name="laser_controller" filename="libgazebo_ros_ray_sensor.so">
                 <ros>
-                    <argument>out:=scan</argument>
+                    <argument>~/out:=scan</argument>
                 </ros>
                 <output_type>sensor_msgs/LaserScan</output_type>
-                <frame_name>laser_frame</frame_name>
+                <frame_name>lidar_link</frame_name>
             </plugin>
         </sensor>

File: description/properties.xacro (robot description, xacro)
@@ -19,7 +19,7 @@
     <xacro:property name="camera_height" value="0.050"/>
     <xacro:property name="camera_mass" value="0.250"/>
-    <xacro:property name="hokuyo_base" value="0.1"/>
-    <xacro:property name="hokuyo_mass" value="0.1"/>
-    <xacro:property name="hokuyo_radius" value="0.05"/>
+    <xacro:property name="lidar_base" value="0.1"/>
+    <xacro:property name="lidar_mass" value="0.1"/>
+    <xacro:property name="lidar_radius" value="0.05"/>
     <material name="white">
         <color rgba="1 1 1 1" />

File: description/robotie.xacro (robot description, xacro)
@@ -118,12 +118,12 @@
         </collision>
     </link>
-    <!--HOKUYO_LASER-->
-    <joint name="hokuyo_base_joint" type="fixed">
+    <!--LIDAR-->
+    <joint name="lidar_base_joint" type="fixed">
         <origin xyz="${chassis_length/2} 0.0 ${chassis_height}" rpy="0.0 0.0 0.0"/>
         <parent link="chassis"/>
-        <child link="hokuyo_base_link"/>
+        <child link="lidar_base_link"/>
     </joint>
-    <link name="hokuyo_base_link">
-        <xacro:inertial_box mass="${hokuyo_mass}" x="${hokuyo_base}" y="${hokuyo_base}" z="${hokuyo_base}">
+    <link name="lidar_base_link">
+        <xacro:inertial_box mass="${lidar_mass}" x="${lidar_base}" y="${lidar_base}" z="${lidar_base}">
             <origin xyz="0.0 0.0 0.0" rpy="0.0 0.0 0.0"/>
         </xacro:inertial_box>
@@ -131,5 +131,5 @@
             <origin xyz="0.0 0.0 0.0" rpy="0.0 0.0 0.0"/>
             <geometry>
-                <box size="${hokuyo_base} ${hokuyo_base} ${hokuyo_base/2}"/>
+                <box size="${lidar_base} ${lidar_base} ${lidar_base/2}"/>
             </geometry>
             <material name="black"/>
@@ -138,15 +138,15 @@
             <origin xyz="0.0 0.0 0.0" rpy="0.0 0.0 0.0"/>
             <geometry>
-                <box size="${hokuyo_base} ${hokuyo_base} ${hokuyo_base/2}"/>
+                <box size="${lidar_base} ${lidar_base} ${lidar_base/2}"/>
             </geometry>
         </collision>
     </link>
-    <joint name="hokuyo_joint" type="fixed">
-        <origin xyz="0.0 0.0 ${hokuyo_base/4}" rpy="0.0 0.0 0.0"/>
-        <parent link="hokuyo_base_link"/>
-        <child link="hokuyo_link"/>
+    <joint name="lidar_joint" type="fixed">
+        <origin xyz="0.0 0.0 ${lidar_base/4}" rpy="0.0 0.0 0.0"/>
+        <parent link="lidar_base_link"/>
+        <child link="lidar_link"/>
     </joint>
-    <link name="hokuyo_link">
-        <xacro:inertial_cylinder mass="${hokuyo_mass}" length="${hokuyo_base}" radius="${hokuyo_radius}">
+    <link name="lidar_link">
+        <xacro:inertial_cylinder mass="${lidar_mass}" length="${lidar_base}" radius="${lidar_radius}">
             <origin xyz="0 0 0" rpy="0 0 0"/>
         </xacro:inertial_cylinder>
@@ -154,5 +154,5 @@
             <origin xyz="0.0 0.0 0.0" rpy="0.0 0.0 0.0"/>
             <geometry>
-                <cylinder radius="${hokuyo_radius}" length="${hokuyo_base}"/>
+                <cylinder radius="${lidar_radius}" length="${lidar_base}"/>
             </geometry>
             <material name="black"/>
@@ -161,5 +161,5 @@
             <origin xyz="0.0 0.0 0.0" rpy="0.0 0.0 0.0"/>
             <geometry>
-                <cylinder radius="${hokuyo_radius}" length="${hokuyo_base}"/>
+                <cylinder radius="${lidar_radius}" length="${lidar_base}"/>
             </geometry>
         </collision>

Commit message: nav2_integration

File: description/gazebo.xacro (robot description, xacro)
@@ -61,4 +61,5 @@
         </sensor>
     </gazebo>
+    <!--LIDAR-->
     <gazebo reference="lidar_base_link">
         <material>

File: description/properties.xacro (robot description, xacro)
@@ -5,5 +5,5 @@
     <xacro:property name="chassis_height" value="0.138"/>
     <xacro:property name="chassis_mass" value="1.0"/>
-    <xacro:property name="wheel_radius" value="0.05"/>
+    <xacro:property name="wheel_radius" value="0.033"/>
     <xacro:property name="wheel_thickness" value="0.026"/>
     <xacro:property name="wheel_mass" value="0.05"/>

File: description/ros2_control.xacro (robot description, xacro)
@@ -7,6 +7,6 @@
         <joint name="left_wheel_joint">
             <command_interface name="velocity">
-                <param name="min">-0.1</param>
-                <param name="max">1</param>
+                <param name="min">-10</param>
+                <param name="max">10</param>
             </command_interface>
             <state_interface name="velocity"/>
@@ -15,6 +15,6 @@
          <joint name="right_wheel_joint">
             <command_interface name="velocity">
-                <param name="min">-0.1</param>
-                <param name="max">1</param>
+                <param name="min">-10</param>
+                <param name="max">10</param>
             </command_interface>
             <state_interface name="velocity"/>

Commit message: ackermann_steering

File: description/gazebo.xacro (robot description, xacro)
@@ -6,5 +6,5 @@
         </material>
     </gazebo>
-    <gazebo reference="left_wheel">
+    <gazebo reference="left_wheel_back">
         <material>
             Gazebo/Black
@@ -13,5 +13,5 @@
         <mu2>0.2</mu2>
     </gazebo>
-    <gazebo reference="right_wheel">
+    <gazebo reference="right_wheel_back">
         <material>
             Gazebo/Black
@@ -20,5 +20,19 @@
         <mu2>0.2</mu2>
     </gazebo>
-    <gazebo reference="caster_wheel">
+    <gazebo reference="left_wheel_front">
+        <material>
+            Gazebo/Black
+        </material>
+        <mu1>0.2</mu1>
+        <mu2>0.2</mu2>
+    </gazebo>
+    <gazebo reference="right_wheel_front">
+        <material>
+            Gazebo/Black
+        </material>
+        <mu1>0.2</mu1>
+        <mu2>0.2</mu2>
+    </gazebo>
+    <!-- <gazebo reference="caster_wheel">
         <material>
             Gazebo/Black
@@ -26,5 +40,5 @@
         <mu1>0.02</mu1>
         <mu2>0.02</mu2>
-    </gazebo>
+    </gazebo> -->
     <!--CAMERA_PLUGIN-->
     <gazebo reference="camera_link">

File: description/properties.xacro (robot description, xacro)
@@ -1,12 +1,13 @@
 <?xml version="1.0"?>
 <robot xmlns:xacro="http://www.ros.org/wiki/xacro">
-    <xacro:property name="chassis_length" value="0.335"/>
+    <xacro:property name="chassis_length" value="0.45"/>
     <xacro:property name="chassis_width" value="0.265"/>
     <xacro:property name="chassis_height" value="0.138"/>
     <xacro:property name="chassis_mass" value="1.0"/>
-    <xacro:property name="wheel_radius" value="0.033"/>
+    <xacro:property name="wheel_radius" value="0.05"/>
     <xacro:property name="wheel_thickness" value="0.026"/>
     <xacro:property name="wheel_mass" value="0.05"/>
-    <xacro:property name="wheel_offset_x" value="0.226"/>
+    <xacro:property name="wheel_offset_x" value="0.1"/>
+    <xacro:property name="wheel_offset_x_front" value="0.25"/>
     <xacro:property name="wheel_offset_y" value="0.1485"/>
     <xacro:property name="wheel_offset_z" value="0.01"/>

File: description/robotie.xacro (robot description, xacro)
@@ -36,11 +36,12 @@
         </xacro:inertial_box>
     </link>
-    <joint name="left_wheel_joint" type="continuous">
+    <!--BACK-->
+    <joint name="left_wheel_joint_back" type="continuous">
         <parent link="base_link"/>
-        <child link="left_wheel"/>
+        <child link="left_wheel_back"/>
         <origin xyz="0 ${wheel_offset_y} 0" rpy="-${pi/2} 0 0" />
         <axis xyz="0 0 1"/>
     </joint>
-    <link name="left_wheel">
+    <link name="left_wheel_back">
         <visual>
             <geometry>
@@ -58,11 +59,11 @@
         </xacro:inertial_cylinder>
     </link>
-    <joint name="right_wheel_joint" type="continuous">
+    <joint name="right_wheel_joint_back" type="continuous">
         <parent link="base_link"/>
-        <child link="right_wheel"/>
+        <child link="right_wheel_back"/>
         <origin xyz="0 ${-wheel_offset_y} 0" rpy="${pi/2} 0 0" />
         <axis xyz="0 0 -1"/>
     </joint>
-    <link name="right_wheel">
+    <link name="right_wheel_back">
         <visual>
             <geometry>
@@ -80,13 +81,15 @@
         </xacro:inertial_cylinder>
     </link>
-    <joint name="caster_wheel_joint" type="fixed">
-        <parent link="chassis"/>
-        <child link="caster_wheel"/>
-        <origin xyz="${caster_wheel_offset_x} 0 ${caster_wheel_offset_z}"/>
+    <!--FRONT-->
+    <joint name="left_wheel_joint_front" type="continuous">
+        <parent link="base_link"/>
+        <child link="left_wheel_front"/>
+        <origin xyz="${wheel_offset_x_front} ${wheel_offset_y} 0" rpy="-${pi/2} 0 0" />
+        <axis xyz="0 0 1"/>
     </joint>
-    <link name="caster_wheel">
+    <link name="left_wheel_front">
         <visual>
             <geometry>
-                <sphere radius="${caster_wheel_radius}"/>
+                <cylinder radius="${wheel_radius}" length="${wheel_thickness}"/>
             </geometry>
             <material name="black"/>
@@ -94,10 +97,32 @@
         <collision>
             <geometry>
-                <sphere radius="${caster_wheel_radius}"/>
+                <sphere radius="${wheel_radius}"/>
             </geometry>
         </collision>
-        <xacro:inertial_sphere mass="${caster_wheel_mass}" radius="${caster_wheel_radius}">
+        <xacro:inertial_cylinder mass="${wheel_mass}" length="${wheel_thickness}" radius="${wheel_radius}">
             <origin xyz="0 0 0" rpy="0 0 0"/>
-        </xacro:inertial_sphere>
+        </xacro:inertial_cylinder>
+    </link>
+    <joint name="right_wheel_joint_front" type="continuous">
+        <parent link="base_link"/>
+        <child link="right_wheel_front"/>
+        <origin xyz="${wheel_offset_x_front} ${-wheel_offset_y} 0" rpy="${pi/2} 0 0" />
+        <axis xyz="0 0 -1"/>
+    </joint>
+    <link name="right_wheel_front">
+        <visual>
+            <geometry>
+                <cylinder radius="${wheel_radius}" length="${wheel_thickness}"/>
+            </geometry>
+            <material name="black"/>
+        </visual>
+        <collision>
+            <geometry>
+                <sphere radius="${wheel_radius}"/>
+            </geometry>
+        </collision>
+        <xacro:inertial_cylinder mass="${wheel_mass}" length="${wheel_thickness}" radius="${wheel_radius}">
+            <origin xyz="0 0 0" rpy="0 0 0"/>
+        </xacro:inertial_cylinder>
     </link>
     <!--CAMERA-->

File: description/ros2_control.xacro (robot description, xacro)
@@ -5,5 +5,5 @@
             <plugin>gazebo_ros2_control/GazeboSystem</plugin>
         </hardware>
-        <joint name="left_wheel_joint">
+        <joint name="left_wheel_joint_front">
             <command_interface name="velocity">
                 <param name="min">-10</param>
@@ -13,5 +13,5 @@
             <state_interface name="position"/>
         </joint>
-         <joint name="right_wheel_joint">
+         <joint name="right_wheel_joint_front">
             <command_interface name="velocity">
                 <param name="min">-10</param>
